File: CapKeys.kicad_sch (KiCad schematic)
At the start: 97 parts, among them J1 USB_C_Receptacle_USB2.0_16P, J19 Conn_01x01, J20 Conn_01x01, U1 W25Q128JVS, U2 MPR121QR2, U3 AMS1117-3.3, U4 MPR121QR2, U5 MPR121QR2, U6 MPR121QR2, U7 RP2040, Y1 X322512MSB4SI

Commit message: Updated PCB
Parts:
- U7: footprint Package_DFN_QFN:QFN-56-1EP_7x7mm_P0.4mm_EP3.2x3.2mm -> Package_DFN_QFN:QFN-56-1EP_7x7mm_P0.4mm_EP3.2x3.2mm_ThermalVias
Changed lines of the file:
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@@
 			)
 		)
-		(property "Footprint" "Package_DFN_QFN:QFN-56-1EP_7x7mm_P0.4mm_EP3.2x3.2mm"
+		(property "Footprint" "Package_DFN_QFN:QFN-56-1EP_7x7mm_P0.4mm_EP3.2x3.2mm_ThermalVias"
 			(at 355.6 95.25 0)
 			(hide yes)
