File: CapKeys.kicad_pcb (KiCad board)
At the start: 4 copper layers, 215 x 130 mm, 101 parts, among them J1 USB_C_Receptacle_USB2.0_16P, J19 Conn_01x01, J20 Conn_01x01, U1 W25Q128JVS, U2 MPR121QR2, U3 AMS1117-3.3, U4 MPR121QR2, U5 MPR121QR2, U6 MPR121QR2, U7 RP2040, Y1 X322512MSB4SI

Commit message: Updated PCB
Parts:
- removed H3, H4, H5, H6: MountingHole, MountingHole:MountingHole_3.2mm_M3
- moved H2 215.0 mm to (309.0, 111.0)
- moved H1 31.0 mm to (106.0, 111.0)
Routing:
- net /LED_PTB-2: track 0.00 -> 166.5 mm, vias 0 -> 2
- net /KEY_A_1: track 0.00 -> 127.6 mm, vias 0 -> 2
- net /KEY_HC_1: track 0.00 -> 114.0 mm, vias 0 -> 2
- net /KEY_F_1: track 0.00 -> 111.6 mm, vias 0 -> 2
- net /KEY_E_1: track 0.00 -> 109.2 mm, vias 0 -> 2
- net /KEY_G_1: track 0.00 -> 108.6 mm, vias 0 -> 2
- net /KEY_B_1: track 0.00 -> 107.3 mm, vias 0 -> 2
- net /KEY_D_1: track 0.00 -> 99.4 mm, vias 0 -> 3
- net /KEY_D_2: track 0.00 -> 98.5 mm, vias 0 -> 2
- net /KEY_G_2: track 0.00 -> 97.7 mm, vias 0 -> 2
- net /KEY_HC_2: track 0.00 -> 93.9 mm, vias 0 -> 2
- net /KEY_A_2: track 0.00 -> 89.7 mm, vias 0 -> 2
- net /KEY_F_2: track 0.00 -> 89.4 mm, vias 0 -> 2
- net /KEY_D#_1: track 0.00 -> 84.4 mm, vias 0 -> 2
- net /KEY_B_2: track 0.00 -> 83.9 mm, vias 0 -> 2
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
Commit message: Updated PCB and Footprints
Parts:
- U2, U4, U5, U6: footprint Footprints:QFN40P300X300X60-20N -> Package_DFN_QFN:UQFN-20_3x3mm_P0.4mm
- U7: footprint Package_DFN_QFN:QFN-56-1EP_7x7mm_P0.4mm_EP3.2x3.2mm -> Package_DFN_QFN:QFN-56-1EP_7x7mm_P0.4mm_EP3.2x3.2mm_ThermalVias
- moved U6 0.06 mm to (262.6, 131.0)
Routing:
- net /KEY_D_1: track 99.4 -> 114.7 mm, vias 3 -> 2
- net VBUS: track 85.9 -> 71.4 mm
- net /LED_PTB-2: track 166.5 -> 155.3 mm
- net /SDA: track 194.1 -> 185.7 mm, vias 5 -> 6
- net /KEY_A_1: track 127.6 -> 135.3 mm
- net /KEY_A_2: track 89.7 -> 97.0 mm
- net GND: track 36.8 -> 43.9 mm, vias 132 -> 119
- net +3V3: track 72.1 -> 78.1 mm, vias 46 -> 44
- net /RUN: track 1.76 -> 6.70 mm
- net /KEY_C#_3: track 70.2 -> 68.0 mm, vias 3 -> 2
- net /SCL: track 182.4 -> 184.0 mm
- net /LED_HC: track 150.3 -> 148.7 mm
- net Net-(J1-CC2): track 6.21 -> 7.18 mm
- net /LED_A#: track 116.9 -> 117.7 mm
- net Net-(J1-CC1): track 7.13 -> 7.79 mm
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
Commit message: Updated PCB
Routing:
- net /LED_F: track 58.2 -> 63.1 mm
- net /LED_B: track 132.5 -> 135.7 mm
- net /LED_HC: track 148.7 -> 151.8 mm
- net /LED_A: track 108.6 -> 110.2 mm
- net /LED_G: track 84.6 -> 85.6 mm
- net /KEY_B_2: track 83.9 -> 84.7 mm
- net /KEY_B_1: track 107.3 -> 107.8 mm
- net GND: vias 119 -> 145
- net +3V3: vias 44 -> 50
Other:
- board text added: "CapKeys"
